File: pcbkicad/pcbkicad.sch (KiCad schematic (older format))
At the start: 35 parts, among them J1 USBDaughterboard, U1 AMS1117-3.3, U2 STM32F072CBTx

Commit message: Schematic protection
Parts:
- removed J1: USBDaughterboard, random-keyboard-parts:Molex-0548190589, symbol Connector_Generic:Conn_01x04
- added D?: D_TVS, symbol Device:D_TVS
- added F?: 500 mA, symbol Device:Fuse
- added J?: USB_C_Receptacle_USB2.0, symbol Connector:USB_C_Receptacle_USB2.0
- added R? (x2): 5.1k, symbol Device:R_Small_US
- added U?: TPD4E02B04DQA, Package_SON:USON-10_2.5x1.0mm_P0.5mm, symbol Power_Protection:TPD4E02B04DQA
Connections:
- net labels added: GNDPWR
- wire segments 106 -> 128
Changed lines of the file:
@@
 BOOT0
 Wire Wire Line
-	5250 1900 5450 1900
+	5250 1900 5350 1900
 Wire Wire Line
 	5450 1900 5450 2050
@@
 	850  3500 1350 3500
 Connection ~ 1350 3500
-$Comp
-L Connector_Generic:Conn_01x04 J1
-U 1 1 5FC96AD3
-P 8950 3400
-F 0 "J1" H 9030 3392 50  0000 L CNN
-F 1 "USBDaughterboard" H 9030 3301 50  0000 L CNN
-F 2 "random-keyboard-parts:Molex-0548190589" H 8950 3400 50  0001 C CNN
-F 3 "~" H 8950 3400 50  0001 C CNN
-	1    8950 3400
-	1    0    0    -1
-$EndComp
-Wire Wire Line
-	8750 3300 8600 3300
-Wire Wire Line
-	8600 3300 8600 3200
-$Comp
-L power:VCC #PWR0111
-U 1 1 5FC9F18A
-P 8600 3200
-F 0 "#PWR0111" H 8600 3050 50  0001 C CNN
-F 1 "VCC" H 8615 3373 50  0000 C CNN
-F 2 "" H 8600 3200 50  0001 C CNN
-F 3 "" H 8600 3200 50  0001 C CNN
-	1    8600 3200
-	1    0    0    -1
-$EndComp
-$Comp
-L power:GND #PWR0112
-U 1 1 5FCA0124
-P 8600 3700
-F 0 "#PWR0112" H 8600 3450 50  0001 C CNN
-F 1 "GND" H 8605 3527 50  0000 C CNN
-F 2 "" H 8600 3700 50  0001 C CNN
-F 3 "" H 8600 3700 50  0001 C CNN
-	1    8600 3700
-	1    0    0    -1
-$EndComp
-Wire Wire Line
-	8750 3600 8600 3600
-Wire Wire Line
-	8600 3600 8600 3700
-Text GLabel 8450 3400 0    50   Input ~ 0
-D-
-Text GLabel 8450 3500 0    50   Input ~ 0
-D+
-Wire Wire Line
-	8450 3500 8750 3500
-Wire Wire Line
-	8450 3400 8750 3400
 $Comp
 L MX_Alps_Hybrid:MX-NoLED MX1
@@
 	5550 5050 5350 5050
 Wire Wire Line
-	5350 2050 5350 1750
-Wire Wire Line
 	5350 1750 5750 1750
 Wire Wire Line
@@
 L power:VCC #PWR0101
 U 1 1 5FC3DB8A
-P 1950 1250
-F 0 "#PWR0101" H 1950 1100 50  0001 C CNN
-F 1 "VCC" H 1965 1423 50  0000 C CNN
-F 2 "" H 1950 1250 50  0001 C CNN
-F 3 "" H 1950 1250 50  0001 C CNN
-	1    1950 1250
-	1    0    0    -1
-$EndComp
-Wire Wire Line
-	1950 1250 1950 1400
-Wire Wire Line
-	1950 1400 2200 1400
+P 1000 1250
+F 0 "#PWR0101" H 1000 1100 50  0001 C CNN
+F 1 "VCC" H 1015 1423 50  0000 C CNN
+F 2 "" H 1000 1250 50  0001 C CNN
+F 3 "" H 1000 1250 50  0001 C CNN
+	1    1000 1250
+	1    0    0    -1
+$EndComp
+Wire Wire Line
+	1000 1250 1000 1400
+Wire Wire Line
+	1000 1400 1250 1400
+$Comp
+L Connector:USB_C_Receptacle_USB2.0 J?
+U 1 1 5FC3F0C4
+P 1700 6150
+F 0 "J?" H 1807 7017 50  0000 C CNN
+F 1 "USB_C_Receptacle_USB2.0" H 1807 6926 50  0000 C CNN
+F 2 "" H 1850 6150 50  0001 C CNN
+F 3 "https://www.usb.org/sites/default/files/documents/usb_type-c.zip" H 1850 6150 50  0001 C CNN
+	1    1700 6150
+	1    0    0    -1
+$EndComp
+$Comp
+L Power_Protection:TPD4E02B04DQA U?
+U 1 1 5FC3FDD9
+P 3100 6200
+F 0 "U?" V 3525 6250 50  0000 C CNN
+F 1 "TPD4E02B04DQA" V 3434 6250 50  0000 C CNN
+F 2 "Package_SON:USON-10_2.5x1.0mm_P0.5mm" H 3400 6200 50  0001 L CNN
+F 3 "http://www.ti.com/lit/ds/symlink/tpd4e02b04.pdf" H 3225 6525 50  0001 C CNN
+	1    3100 6200
+	0    -1   -1   0
+$EndComp
+Wire Wire Line
+	2300 6050 2600 6050
+Wire Wire Line
+	2800 6050 2800 6000
+Wire Wire Line
+	2300 6150 2600 6150
+Wire Wire Line
+	2800 6150 2800 6100
+Wire Wire Line
+	2800 6250 2800 6300
+Wire Wire Line
+	2300 6350 2500 6350
+Wire Wire Line
+	2800 6350 2800 6400
+$Comp
+L power:GNDPWR #PWR?
+U 1 1 5FC56B0E
+P 3450 6300
+F 0 "#PWR?" H 3450 6100 50  0001 C CNN
+F 1 "GNDPWR" H 3454 6146 50  0000 C CNN
+F 2 "" H 3450 6250 50  0001 C CNN
+F 3 "" H 3450 6250 50  0001 C CNN
+	1    3450 6300
+	1    0    0    -1
+$EndComp
+Wire Wire Line
+	3450 6300 3450 6200
+Wire Wire Line
+	3450 6200 3300 6200
+$Comp
+L power:GNDPWR #PWR?
+U 1 1 5FC6229C
+P 1700 7050
+F 0 "#PWR?" H 1700 6850 50  0001 C CNN
+F 1 "GNDPWR" H 1704 6896 50  0000 C CNN
+F 2 "" H 1700 7000 50  0001 C CNN
+F 3 "" H 1700 7000 50  0001 C CNN
+	1    1700 7050
+	1    0    0    -1
+$EndComp
+$Comp
+L power:GNDPWR #PWR?
+U 1 1 5FC633A4
+P 1400 7050
+F 0 "#PWR?" H 1400 6850 50  0001 C CNN
+F 1 "GNDPWR" H 1404 6896 50  0000 C CNN
+F 2 "" H 1400 7000 50  0001 C CNN
+F 3 "" H 1400 7000 50  0001 C CNN
+	1    1400 7050
+	1    0    0    -1
+$EndComp
+Wire Wire Line
+	2300 5550 2450 5550
+Wire Wire Line
+	2450 5550 2450 5450
+$Comp
+L power:VCC #PWR?
+U 1 1 5FC687B2
+P 2450 5450
+F 0 "#PWR?" H 2450 5300 50  0001 C CNN
+F 1 "VCC" H 2465 5623 50  0000 C CNN
+F 2 "" H 2450 5450 50  0001 C CNN
+F 3 "" H 2450 5450 50  0001 C CNN
+	1    2450 5450
+	1    0    0    -1
+$EndComp
+Wire Wire Line
+	2600 6050 2600 6150
+Connection ~ 2600 6050
+Wire Wire Line
+	2600 6050 2800 6050
+Connection ~ 2600 6150
+Wire Wire Line
+	2600 6150 2800 6150
+Wire Wire Line
+	2600 6150 2600 6700
+Wire Wire Line
+	2600 6700 2650 6700
+Text GLabel 2650 6700 2    50   Input ~ 0
+D-
+Wire Wire Line
+	2300 6250 2500 6250
+Wire Wire Line
+	2500 6250 2500 6350
+Connection ~ 2500 6250
+Wire Wire Line
+	2500 6250 2800 6250
+Connection ~ 2500 6350
+Wire Wire Line
+	2500 6350 2800 6350
+Wire Wire Line
+	2500 6350 2500 6800
+Wire Wire Line
+	2500 6800 2650 6800
+Text GLabel 2650 6800 2    50   Input ~ 0
+D+
+$Comp
+L Device:Fuse F?
+U 1 1 5FC88487
+P 1400 1400
+F 0 "F?" V 1203 1400 50  0000 C CNN
+F 1 "500 mA" V 1294 1400 50  0000 C CNN
+F 2 "" V 1330 1400 50  0001 C CNN
+F 3 "~" H 1400 1400 50  0001 C CNN
+	1    1400 1400
+	0    1    1    0
+$EndComp
+$Comp
+L Device:D_TVS D?
+U 1 1 5FC8CAA2
+P 1700 1550
+F 0 "D?" V 1654 1630 50  0000 L CNN
+F 1 "D_TVS" V 1745 1630 50  0000 L CNN
+F 2 "" H 1700 1550 50  0001 C CNN
+F 3 "~" H 1700 1550 50  0001 C CNN
+	1    1700 1550
+	0    1    1    0
+$EndComp
+Wire Wire Line
+	1550 1400 1700 1400
+Wire Wire Line
+	1700 1400 2200 1400
+Connection ~ 1700 1400
 Connection ~ 2200 1400
+Wire Wire Line
+	5350 1750 5350 1900
+Connection ~ 5350 1900
+Wire Wire Line
+	5350 1900 5450 1900
+$Comp
+L Device:R_Small_US R?
+U 1 1 5FCA621E
+P 2400 5850
+F 0 "R?" V 2400 6000 50  0000 C CNN
+F 1 "5.1k" V 2500 5900 50  0000 C CNN
+F 2 "" H 2400 5850 50  0001 C CNN
+F 3 "~" H 2400 5850 50  0001 C CNN
+	1    2400 5850
+	0    1    1    0
+$EndComp
+$Comp
+L Device:R_Small_US R?
+U 1 1 5FCA6D1A
+P 2400 5750
+F 0 "R?" V 2195 5750 50  0000 C CNN
+F 1 "5.1k" V 2286 5750 50  0000 C CNN
+F 2 "" H 2400 5750 50  0001 C CNN
+F 3 "~" H 2400 5750 50  0001 C CNN
+	1    2400 5750
+	0    1    1    0
+$EndComp
+Wire Wire Line
+	2500 5750 2650 5750
+Wire Wire Line
+	2650 5750 2650 5850
+Wire Wire Line
+	2650 5850 2500 5850
+Connection ~ 2650 5850
+$Comp
+L power:GNDPWR #PWR?
+U 1 1 5FCB2582
+P 2650 5850
+F 0 "#PWR?" H 2650 5650 50  0001 C CNN
+F 1 "GNDPWR" H 2654 5696 50  0000 C CNN
+F 2 "" H 2650 5800 50  0001 C CNN
+F 3 "" H 2650 5800 50  0001 C CNN
+	1    2650 5850
+	1    0    0    -1
+$EndComp
+$Comp
+L power:GNDPWR #PWR?
+U 1 1 5FCB3671
+P 1700 1700
+F 0 "#PWR?" H 1700 1500 50  0001 C CNN
+F 1 "GNDPWR" H 1704 1546 50  0000 C CNN
+F 2 "" H 1700 1650 50  0001 C CNN
+F 3 "" H 1700 1650 50  0001 C CNN
+	1    1700 1700
+	1    0    0    -1
+$EndComp
 $EndSCHEMATC

Commit message: I honestly don't remember
Parts:
- D1: renamed from D?; footprint (none) -> Diode_SMD:D_0201_0603Metric
- F1: renamed from F?; footprint (none) -> Fuse:Fuse_0402_1005Metric
- J1: renamed from J?; footprint (none) -> Connector_USB:USB_C_Receptacle_HRO_TYPE-C-31-M-12
- R3, R4: renamed from R?; footprint (none) -> Resistor_SMD:R_0805_2012Metric
- gave numbers to parts that had none: 1
Connections:
- wire segments 128 -> 129
Changed lines of the file:
@@
 	1000 1400 1250 1400
 $Comp
-L Connector:USB_C_Receptacle_USB2.0 J?
+L Connector:USB_C_Receptacle_USB2.0 J1
 U 1 1 5FC3F0C4
 P 1700 6150
-F 0 "J?" H 1807 7017 50  0000 C CNN
+F 0 "J1" H 1807 7017 50  0000 C CNN
 F 1 "USB_C_Receptacle_USB2.0" H 1807 6926 50  0000 C CNN
-F 2 "" H 1850 6150 50  0001 C CNN
+F 2 "Connector_USB:USB_C_Receptacle_HRO_TYPE-C-31-M-12" H 1850 6150 50  0001 C CNN
 F 3 "https://www.usb.org/sites/default/files/documents/usb_type-c.zip" H 1850 6150 50  0001 C CNN
 	1    1700 6150
@@
 $EndComp
 $Comp
-L Power_Protection:TPD4E02B04DQA U?
+L Power_Protection:TPD4E02B04DQA U3
 U 1 1 5FC3FDD9
 P 3100 6200
-F 0 "U?" V 3525 6250 50  0000 C CNN
+F 0 "U3" V 3525 6250 50  0000 C CNN
 F 1 "TPD4E02B04DQA" V 3434 6250 50  0000 C CNN
 F 2 "Package_SON:USON-10_2.5x1.0mm_P0.5mm" H 3400 6200 50  0001 L CNN
@@
 	2300 6050 2600 6050
 Wire Wire Line
-	2800 6050 2800 6000
-Wire Wire Line
 	2300 6150 2600 6150
 Wire Wire Line
@@
 Wire Wire Line
 	2300 6350 2500 6350
-Wire Wire Line
-	2800 6350 2800 6400
-$Comp
-L power:GNDPWR #PWR?
+$Comp
+L power:GNDPWR #PWR0108
 U 1 1 5FC56B0E
 P 3450 6300
-F 0 "#PWR?" H 3450 6100 50  0001 C CNN
+F 0 "#PWR0108" H 3450 6100 50  0001 C CNN
 F 1 "GNDPWR" H 3454 6146 50  0000 C CNN
 F 2 "" H 3450 6250 50  0001 C CNN
@@
 	3450 6200 3300 6200
 $Comp
-L power:GNDPWR #PWR?
+L power:GNDPWR #PWR0111
 U 1 1 5FC6229C
 P 1700 7050
-F 0 "#PWR?" H 1700 6850 50  0001 C CNN
+F 0 "#PWR0111" H 1700 6850 50  0001 C CNN
 F 1 "GNDPWR" H 1704 6896 50  0000 C CNN
 F 2 "" H 1700 7000 50  0001 C CNN
@@
 $EndComp
 $Comp
-L power:GNDPWR #PWR?
+L power:GNDPWR #PWR0112
 U 1 1 5FC633A4
 P 1400 7050
-F 0 "#PWR?" H 1400 6850 50  0001 C CNN
+F 0 "#PWR0112" H 1400 6850 50  0001 C CNN
 F 1 "GNDPWR" H 1404 6896 50  0000 C CNN
 F 2 "" H 1400 7000 50  0001 C CNN
@@
 	2450 5550 2450 5450
 $Comp
-L power:VCC #PWR?
+L power:VCC #PWR0115
 U 1 1 5FC687B2
 P 2450 5450
-F 0 "#PWR?" H 2450 5300 50  0001 C CNN
+F 0 "#PWR0115" H 2450 5300 50  0001 C CNN
 F 1 "VCC" H 2465 5623 50  0000 C CNN
 F 2 "" H 2450 5450 50  0001 C CNN
@@
 Wire Wire Line
 	2600 6050 2600 6150
-Connection ~ 2600 6050
-Wire Wire Line
-	2600 6050 2800 6050
 Connection ~ 2600 6150
 Wire Wire Line
 	2600 6150 2800 6150
 Wire Wire Line
-	2600 6150 2600 6700
+	2600 6150 2600 6400
 Wire Wire Line
 	2600 6700 2650 6700
@@
 Connection ~ 2500 6350
 Wire Wire Line
-	2500 6350 2800 6350
-Wire Wire Line
 	2500 6350 2500 6800
 Wire Wire Line
@@
 D+
 $Comp
-L Device:Fuse F?
+L Device:Fuse F1
 U 1 1 5FC88487
 P 1400 1400
-F 0 "F?" V 1203 1400 50  0000 C CNN
+F 0 "F1" V 1203 1400 50  0000 C CNN
 F 1 "500 mA" V 1294 1400 50  0000 C CNN
-F 2 "" V 1330 1400 50  0001 C CNN
+F 2 "Fuse:Fuse_0402_1005Metric" V 1330 1400 50  0001 C CNN
 F 3 "~" H 1400 1400 50  0001 C CNN
 	1    1400 1400
@@
 $EndComp
 $Comp
-L Device:D_TVS D?
+L Device:D_TVS D1
 U 1 1 5FC8CAA2
 P 1700 1550
-F 0 "D?" V 1654 1630 50  0000 L CNN
+F 0 "D1" V 1654 1630 50  0000 L CNN
 F 1 "D_TVS" V 1745 1630 50  0000 L CNN
-F 2 "" H 1700 1550 50  0001 C CNN
+F 2 "Diode_SMD:D_0201_0603Metric" H 1700 1550 50  0001 C CNN
 F 3 "~" H 1700 1550 50  0001 C CNN
 	1    1700 1550
@@
 	5350 1900 5450 1900
 $Comp
-L Device:R_Small_US R?
+L Device:R_Small_US R4
 U 1 1 5FCA621E
 P 2400 5850
-F 0 "R?" V 2400 6000 50  0000 C CNN
+F 0 "R4" V 2400 6000 50  0000 C CNN
 F 1 "5.1k" V 2500 5900 50  0000 C CNN
-F 2 "" H 2400 5850 50  0001 C CNN
+F 2 "Resistor_SMD:R_0805_2012Metric" H 2400 5850 50  0001 C CNN
 F 3 "~" H 2400 5850 50  0001 C CNN
 	1    2400 5850
@@
 $EndComp
 $Comp
-L Device:R_Small_US R?
+L Device:R_Small_US R3
 U 1 1 5FCA6D1A
 P 2400 5750
-F 0 "R?" V 2195 5750 50  0000 C CNN
+F 0 "R3" V 2195 5750 50  0000 C CNN
 F 1 "5.1k" V 2286 5750 50  0000 C CNN
-F 2 "" H 2400 5750 50  0001 C CNN
+F 2 "Resistor_SMD:R_0805_2012Metric" H 2400 5750 50  0001 C CNN
 F 3 "~" H 2400 5750 50  0001 C CNN
 	1    2400 5750
@@
 Connection ~ 2650 5850
 $Comp
-L power:GNDPWR #PWR?
+L power:GNDPWR #PWR0116
 U 1 1 5FCB2582
 P 2650 5850
-F 0 "#PWR?" H 2650 5650 50  0001 C CNN
+F 0 "#PWR0116" H 2650 5650 50  0001 C CNN
 F 1 "GNDPWR" H 2654 5696 50  0000 C CNN
 F 2 "" H 2650 5800 50  0001 C CNN
@@
 $EndComp
 $Comp
-L power:GNDPWR #PWR?
+L power:GNDPWR #PWR0117
 U 1 1 5FCB3671
 P 1700 1700
-F 0 "#PWR?" H 1700 1500 50  0001 C CNN
+F 0 "#PWR0117" H 1700 1500 50  0001 C CNN
 F 1 "GNDPWR" H 1704 1546 50  0000 C CNN
 F 2 "" H 1700 1650 50  0001 C CNN
@@
 	1    0    0    -1
 $EndComp
+Wire Wire Line
+	2500 6350 2700 6350
+Wire Wire Line
+	2700 6350 2700 6000
+Wire Wire Line
+	2700 6000 2800 6000
+Wire Wire Line
+	2600 6400 2800 6400
+Connection ~ 2600 6400
+Wire Wire Line
+	2600 6400 2600 6700
 $EndSCHEMATC
